File: schematics/visualizator/visualizator.kicad_pcb (KiCad board)
At the start: 2 copper layers, 48.3 x 43.2 mm, 20 parts, among them J1 5V, J2 WS2812, J3 Audio, SW1 COLOR, SW2 PATTERN, U1 ATmega328-16PU, Y1 16MHz

Commit message: Changed drsign rules
Other:
- net class Default: clearance 1 -> 0.5; via_dia 0.8 -> 1.8; via_drill 0.4 -> 0.6
- rule trace_clearance: 1 -> 0.5
Changed lines of the file:
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@@
   (setup
     (last_trace_width 1)
-    (trace_clearance 1)
+    (trace_clearance 0.5)
     (zone_clearance 1)
     (zone_45_only no)
@@
     (segment_width 0.2)
     (edge_width 0.15)
-    (via_size 0.8)
-    (via_drill 0.4)
+    (via_size 1.8)
+    (via_drill 0.6)
     (via_min_size 0.4)
     (via_min_drill 0.3)
@@
   (net 32 "Net-(R7-Pad2)")
   (net_class Default "This is the default net class."
-    (clearance 1)
+    (clearance 0.5)
     (trace_width 1)
-    (via_dia 0.8)
-    (via_drill 0.4)
+    (via_dia 1.8)
+    (via_drill 0.6)
     (uvia_dia 0.3)
     (uvia_drill 0.1)
@@
   (segment (start 62.23 60.96) (end 66.04 60.96) (width 1) (layer B.Cu) (net 31))
   (segment (start 77.47 57.28863) (end 77.47 58.42) (width 1) (layer B.Cu) (net 32))
+  (segment (start 73.66 50.8) (end 74.79137 50.8) (width 1) (layer B.Cu) (net 32))
   (segment (start 77.47 53.47863) (end 77.47 57.28863) (width 1) (layer B.Cu) (net 32))
   (segment (start 74.79137 50.8) (end 77.47 53.47863) (width 1) (layer B.Cu) (net 32))
-  (segment (start 73.66 50.8) (end 74.79137 50.8) (width 1) (layer B.Cu) (net 32))
   (zone (net 13) (net_name "Net-(C1-Pad1)") (layer B.Cu) (hatch edge 0.508)
     (connect_pads yes (clearance 1))
