File: schematics/visualizator/visualizator.kicad_pcb (KiCad board)
At the start: 2 copper layers, 41.9 x 43.2 mm, 20 parts, among them J1 5V, J2 WS2812, J3 Audio, SW1 COLOR, SW2 PATTERN, U1 ATmega328-16PU, Y1 16MHz

Commit message: PCB updated
Parts:
- moved C2 2.65 mm to (60.8, 54.2)
- moved C3 2.55 mm to (90.3, 48.0)
- moved R2 2.55 mm to (86.5, 48.0)
- moved R5 2.39 mm to (86.9, 35.3)
- moved R1 2.38 mm to (80.1, 58.3)
- moved U1 2.38 mm to (66.1, 35.4)
- moved J3 1.75 mm to (90.7, 41.0)
- moved R4 1.75 mm to (86.9, 39.7)
- moved C4 1.67 mm to (83.3, 43.5)
- moved RV1 1.24 mm to (90.2, 64.8)
- moved J1 0.80 mm to (58.0, 61.0)
- moved J2 0.80 mm to (58.0, 71.1)
- moved R6 0.59 mm to (62.5, 69.1)
- moved R3 0.53 mm to (83.3, 60.9)
- moved RV2 0.52 mm to (83.3, 64.8)
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Routing:
- net Net-(C1-Pad1): track 140.0 -> 132.1 mm
- net Net-(J1-Pad1): track 77.9 -> 74.6 mm
- net Net-(R7-Pad2): track 9.86 -> 6.72 mm
- net Net-(RV1-Pad2): track 35.7 -> 32.7 mm
- net Net-(R6-Pad2): track 4.86 -> 6.75 mm
- net Net-(C1-Pad2): track 14.7 -> 16.6 mm
- net Net-(C2-Pad1): track 13.1 -> 14.9 mm
- net Net-(SW2-Pad1): track 6.56 -> 7.87 mm
- net Net-(R1-Pad1): track 18.7 -> 17.5 mm
- net Net-(SW1-Pad1): track 11.6 -> 12.3 mm
Other:
- board size 41.9 x 43.2 mm -> 39.3 x 43.2 mm

Commit message: Updated PCB
Parts:
- moved C1 2.66 mm to (55.8, 51.6)
- moved Y1 2.09 mm to (57.6, 41.8)
- moved SW1 1.18 mm to (59.6, 36.5)
- moved SW2 0.57 mm to (62.8, 36.5)
- moved J3 0.44 mm to (90.3, 41.0)
Routing:
- net Net-(C1-Pad1): track 132.1 -> 141.7 mm
- net Net-(C1-Pad2): track 16.6 -> 18.1 mm
- net Net-(C2-Pad1): track 14.9 -> 15.8 mm
- net Net-(SW1-Pad1): track 12.3 -> 11.7 mm
- net Net-(J1-Pad1): track 74.6 -> 74.2 mm, vias 2 -> 0
Changed lines of the file:
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@@
     (thickness 1.6)
     (drawings 6)
-    (tracks 116)
+    (tracks 108)
     (zones 0)
     (modules 20)
@@
   )
   (module Connector_Wire:SolderWirePad_1x03_P3.175mm_Drill1mm (layer F.Cu)
-    (at 90.74 40.97 90)
+    (at 90.3 40.97 90)
     (descr "Wire solder connection")
     (tags connector)
@@
   )
   (module Capacitor_THT:C_Disc_D4.3mm_W1.9mm_P5.00mm (layer F.Cu)
-    (at 58.42 52.07)
+    (at 55.8 51.6)
     (descr "C, Disc series, Radial, pin pitch=5.00mm, , diameter*width=4.3*1.9mm^2, Capacitor, http://www.vishay.com/docs/45233/krseries.pdf")
     (tags "C Disc series Radial pin pitch 5.00mm  diameter 4.3mm width 1.9mm Capacitor")
@@
   )
   (module Connector_Wire:SolderWirePad_1x02_P3.81mm_Drill0.8mm (layer F.Cu)
-    (at 58.42 36.53 90)
+    (at 59.6 36.53 90)
     (descr "Wire solder connection")
     (tags connector)
@@
   )
   (module Connector_Wire:SolderWirePad_1x02_P3.81mm_Drill0.8mm (layer F.Cu)
-    (at 62.23 36.53 90)
+    (at 62.8 36.53 90)
     (descr "Wire solder connection")
     (tags connector)
@@
   )
   (module Crystal:Crystal_HC49-4H_Vertical (layer F.Cu)
-    (at 59.69 41.91 270)
+    (at 57.6 41.8 270)
     (descr "Crystal THT HC-49-4H http://5hertz.com/pdfs/04404_D.pdf")
     (tags "THT crystalHC-49-4H")
@@
   (gr_line (start 93.3 30.6) (end 93.3 73.7) (layer Edge.Cuts) (width 0.15))
   (gr_line (start 54 30.5) (end 93.3 30.5) (layer Edge.Cuts) (width 0.15))
-  (segment (start 65.300001 42.220001) (end 66.1 43.02) (width 1) (layer B.Cu) (net 7))
-  (segment (start 65.175999 42.220001) (end 65.300001 42.220001) (width 1) (layer B.Cu) (net 7))
-  (segment (start 62.23 39.274002) (end 65.175999 42.220001) (width 1) (layer B.Cu) (net 7))
-  (segment (start 62.23 36.83) (end 62.23 39.274002) (width 1) (layer B.Cu) (net 7))
-  (segment (start 58.42 36.83) (end 58.42 37.140824) (width 1) (layer B.Cu) (net 9))
-  (segment (start 65.300001 44.760001) (end 66.1 45.56) (width 1) (layer B.Cu) (net 9))
-  (segment (start 65.130003 44.760001) (end 65.300001 44.760001) (width 1) (layer B.Cu) (net 9))
-  (segment (start 58.42 38.049998) (end 65.130003 44.760001) (width 1) (layer B.Cu) (net 9))
-  (segment (start 58.42 36.83) (end 58.42 38.049998) (width 1) (layer B.Cu) (net 9))
-  (via (at 71.1 55.7) (size 1.8) (drill 0.6) (layers F.Cu B.Cu) (net 12))
-  (via (at 68.9 50.6) (size 1.8) (drill 0.6) (layers F.Cu B.Cu) (net 12))
+  (segment (start 62.8 38.52949) (end 62.8 36.53) (width 1) (layer B.Cu) (net 7))
+  (segment (start 62.8 39.844002) (end 62.8 38.52949) (width 1) (layer B.Cu) (net 7))
+  (segment (start 66.1 43.02) (end 65.300001 42.220001) (width 1) (layer B.Cu) (net 7))
+  (segment (start 65.175999 42.220001) (end 62.8 39.844002) (width 1) (layer B.Cu) (net 7))
+  (segment (start 59.6 38.52949) (end 59.6 36.53) (width 1) (layer B.Cu) (net 9))
+  (segment (start 65.271337 44.760001) (end 59.6 39.088664) (width 1) (layer B.Cu) (net 9))
+  (segment (start 65.300001 44.760001) (end 65.271337 44.760001) (width 1) (layer B.Cu) (net 9))
+  (segment (start 59.6 39.088664) (end 59.6 38.52949) (width 1) (layer B.Cu) (net 9))
+  (segment (start 66.1 45.56) (end 65.300001 44.760001) (width 1) (layer B.Cu) (net 9))
   (segment (start 77.47 71.12) (end 71.12 71.12) (width 1) (layer B.Cu) (net 12))
   (segment (start 62.23 71.12) (end 71.12 71.12) (width 1) (layer B.Cu) (net 12))
@@
   (segment (start 57.95 60.96) (end 55.700319 60.960001) (width 1) (layer B.Cu) (net 12))
   (segment (start 71.12 57.092792) (end 71.12 71.12) (width 1) (layer B.Cu) (net 12))
-  (segment (start 71.1 57.072792) (end 71.12 57.092792) (width 1) (layer B.Cu) (net 12))
-  (segment (start 71.1 55.7) (end 71.1 57.072792) (width 1) (layer B.Cu) (net 12))
   (segment (start 71.12 55.72) (end 71.1 55.7) (width 1) (layer B.Cu) (net 12))
   (segment (start 73.72 55.72) (end 71.12 55.72) (width 1) (layer B.Cu) (net 12))
-  (segment (start 68.86 50.64) (end 68.9 50.6) (width 1) (layer B.Cu) (net 12))
-  (segment (start 66.1 50.64) (end 68.86 50.64) (width 1) (layer B.Cu) (net 12))
-  (segment (start 68.9 53.5) (end 71.1 55.7) (width 1) (layer F.Cu) (net 12))
-  (segment (start 68.9 50.6) (end 68.9 53.5) (width 1) (layer F.Cu) (net 12))
   (segment (start 77.47 71.12) (end 83.3 71.12) (width 1) (layer B.Cu) (net 12))
   (segment (start 90.18 71.12) (end 90.2 71.1) (width 1) (layer B.Cu) (net 12))
   (segment (start 83.3 71.12) (end 90.18 71.12) (width 1) (layer B.Cu) (net 12))
+  (segment (start 66.1 50.64) (end 68.24 50.64) (width 1) (layer B.Cu) (net 12))
+  (segment (start 71.12 53.52) (end 71.12 55.72) (width 1) (layer B.Cu) (net 12))
+  (segment (start 68.24 50.64) (end 71.12 53.52) (width 1) (layer B.Cu) (net 12))
+  (segment (start 71.12 55.72) (end 71.12 57.092792) (width 1) (layer B.Cu) (net 12))
   (segment (start 59.717314 64.77) (end 57.95 64.77) (width 1) (layer B.Cu) (net 13))
   (segment (start 60.49 64.77) (end 59.717314 64.77) (width 1) (layer B.Cu) (net 13))
@@
   (segment (start 55.900321 55.900321) (end 57.15 57.15) (width 1) (layer B.Cu) (net 13))
   (segment (start 55.88 55.88) (end 55.900321 55.900321) (width 1) (layer B.Cu) (net 13))
-  (segment (start 71.26 50.64) (end 71.1 50.8) (width 1) (layer B.Cu) (net 13))
-  (segment (start 73.72 50.64) (end 71.26 50.64) (width 1) (layer B.Cu) (net 13))
-  (segment (start 71.1 50.8) (end 71.1 36.999998) (width 1) (layer B.Cu) (net 13))
-  (segment (start 71.1 52.12863) (end 71.1 50.8) (width 1) (layer B.Cu) (net 13))
-  (segment (start 67.23137 53.18) (end 67.25137 53.2) (width 1) (layer B.Cu) (net 13))
-  (segment (start 66.1 53.18) (end 67.23137 53.18) (width 1) (layer B.Cu) (net 13))
-  (segment (start 70.02863 53.2) (end 71.1 52.12863) (width 1) (layer B.Cu) (net 13))
-  (segment (start 67.25137 53.2) (end 70.02863 53.2) (width 1) (layer B.Cu) (net 13))
-  (segment (start 57.25863 52.1) (end 55.88 52.1) (width 1) (layer B.Cu) (net 13))
-  (segment (start 57.28863 52.07) (end 57.25863 52.1) (width 1) (layer B.Cu) (net 13))
-  (segment (start 58.42 52.07) (end 57.28863 52.07) (width 1) (layer B.Cu) (net 13))
   (segment (start 55.88 52.1) (end 55.88 55.88) (width 1) (layer B.Cu) (net 13))
   (segment (start 90.18 58.18) (end 90.34 58.02) (width 1) (layer B.Cu) (net 13))
@@
   (segment (start 90.34 64.61) (end 90.2 64.75) (width 1) (layer B.Cu) (net 13))
   (segment (start 90.34 58.02) (end 90.34 64.61) (width 1) (layer B.Cu) (net 13))
-  (segment (start 71.1 33.12) (end 71.2 33.02) (width 1) (layer B.Cu) (net 13))
-  (segment (start 71.1 36.999998) (end 71.1 33.12) (width 1) (layer B.Cu) (net 13))
   (segment (start 55.88 35.26) (end 58.42 32.72) (width 1) (layer B.Cu) (net 13))
-  (segment (start 55.88 52.1) (end 55.88 35.26) (width 1) (layer B.Cu) (net 13))
   (segment (start 88.972686 37.795) (end 90.74 37.795) (width 1) (layer B.Cu) (net 13))
   (segment (start 81.899002 37.795) (end 88.972686 37.795) (width 1) (layer B.Cu) (net 13))
@@
   (segment (start 83.3 50.7) (end 83.3 54.95) (width 1) (layer B.Cu) (net 13))
   (segment (start 73.72 50.64) (end 83.24 50.64) (width 1) (layer B.Cu) (net 13))
-  (segment (start 65.300001 54.920001) (end 66.1 55.72) (width 1) (layer B.Cu) (net 14))
-  (segment (start 65.138631 54.920001) (end 65.300001 54.920001) (width 1) (layer B.Cu) (net 14))
-  (segment (start 63.42 53.20137) (end 65.138631 54.920001) (width 1) (layer B.Cu) (net 14))
-  (segment (start 63.42 52.07) (end 63.42 53.20137) (width 1) (layer B.Cu) (net 14))
-  (segment (start 63.42 45.64) (end 59.69 41.91) (width 1) (layer B.Cu) (net 14))
-  (segment (start 63.42 52.07) (end 63.42 45.64) (width 1) (layer B.Cu) (net 14))
+  (segment (start 55.88 52.1) (end 55.88 39.5) (width 1) (layer B.Cu) (net 13))
+  (segment (start 55.88 39.5) (end 55.88 35.26) (width 1) (layer B.Cu) (net 13))
+  (segment (start 71.2 33.02) (end 71.1 33.12) (width 1) (layer B.Cu) (net 13))
+  (segment (start 72.26 50.64) (end 73.72 50.64) (width 1) (layer B.Cu) (net 13))
+  (segment (start 72.2 50.7) (end 72.26 50.64) (width 1) (layer B.Cu) (net 13))
+  (segment (start 71.1 33.12) (end 71.1 49.6) (width 1) (layer B.Cu) (net 13))
+  (segment (start 71.1 49.6) (end 72.2 50.7) (width 1) (layer B.Cu) (net 13))
+  (segment (start 57.890002 39.5) (end 55.88 39.5) (width 1) (layer B.Cu) (net 13))
+  (segment (start 66.1 53.18) (end 64.96863 53.18) (width 1) (layer B.Cu) (net 13))
+  (segment (start 63.18863 51.4) (end 63.18863 44.798628) (width 1) (layer B.Cu) (net 13))
+  (segment (start 64.96863 53.18) (end 63.18863 51.4) (width 1) (layer B.Cu) (net 13))
+  (segment (start 63.18863 44.798628) (end 57.890002 39.5) (width 1) (layer B.Cu) (net 13))
+  (segment (start 60.8 45) (end 60.8 51.6) (width 1) (layer B.Cu) (net 14))
+  (segment (start 57.6 41.8) (end 60.8 45) (width 1) (layer B.Cu) (net 14))
+  (segment (start 64.92 55.72) (end 66.1 55.72) (width 1) (layer B.Cu) (net 14))
+  (segment (start 60.8 51.6) (end 64.92 55.72) (width 1) (layer B.Cu) (net 14))
   (segment (start 73.72 48.1) (end 80.1 48.1) (width 1) (layer B.Cu) (net 15))
   (segment (start 86.45 48.1) (end 86.53 48.02) (width 1) (layer B.Cu) (net 15))
@@
   (segment (start 64.86 58.26) (end 66.1 58.26) (width 1) (layer B.Cu) (net 16))
   (segment (start 60.8 54.2) (end 64.86 58.26) (width 1) (layer B.Cu) (net 16))
-  (segment (start 60.8 47.9) (end 59.69 46.79) (width 1) (layer B.Cu) (net 16))
-  (segment (start 60.8 54.2) (end 60.8 47.9) (width 1) (layer B.Cu) (net 16))
+  (segment (start 57.6 51) (end 57.6 46.68) (width 1) (layer B.Cu) (net 16))
+  (segment (start 60.8 54.2) (end 57.6 51) (width 1) (layer B.Cu) (net 16))
   (via (at 76.8 45.5) (size 1.8) (drill 0.6) (layers F.Cu B.Cu) (net 17))
   (via (at 76.8 53) (size 1.8) (drill 0.6) (layers F.Cu B.Cu) (net 17))

Commit message: PCB updated
Parts:
- moved J3 0.37 mm to (90.3, 40.6)
Routing:
- net Net-(C1-Pad1): track 141.7 -> 141.1 mm
- net Net-(J3-Pad1): track 4.34 -> 3.74 mm
Changed lines of the file:
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@@
     (thickness 1.6)
     (drawings 6)
-    (tracks 108)
+    (tracks 107)
     (zones 0)
     (modules 20)
@@
   )
   (module Connector_Wire:SolderWirePad_1x03_P3.175mm_Drill1mm (layer F.Cu)
-    (at 90.3 40.97 90)
+    (at 90.3 40.6 90)
     (descr "Wire solder connection")
     (tags connector)
@@
   (segment (start 90.34 58.02) (end 90.34 64.61) (width 1) (layer B.Cu) (net 13))
   (segment (start 55.88 35.26) (end 58.42 32.72) (width 1) (layer B.Cu) (net 13))
-  (segment (start 88.972686 37.795) (end 90.74 37.795) (width 1) (layer B.Cu) (net 13))
-  (segment (start 81.899002 37.795) (end 88.972686 37.795) (width 1) (layer B.Cu) (net 13))
-  (segment (start 76.824002 32.72) (end 81.899002 37.795) (width 1) (layer B.Cu) (net 13))
   (segment (start 58.42 32.72) (end 76.824002 32.72) (width 1) (layer B.Cu) (net 13))
   (segment (start 83.3 54.95) (end 86.53 58.18) (width 1) (layer B.Cu) (net 13))
@@
   (segment (start 64.96863 53.18) (end 63.18863 51.4) (width 1) (layer B.Cu) (net 13))
   (segment (start 63.18863 44.798628) (end 57.890002 39.5) (width 1) (layer B.Cu) (net 13))
+  (segment (start 81.529002 37.425) (end 90.3 37.425) (width 1) (layer B.Cu) (net 13))
+  (segment (start 76.824002 32.72) (end 81.529002 37.425) (width 1) (layer B.Cu) (net 13))
   (segment (start 60.8 45) (end 60.8 51.6) (width 1) (layer B.Cu) (net 14))
   (segment (start 57.6 41.8) (end 60.8 45) (width 1) (layer B.Cu) (net 14))
@@
   (segment (start 76.74 39.67) (end 76.77 39.7) (width 1) (layer B.Cu) (net 26))
   (segment (start 76.74 35.3) (end 76.74 39.67) (width 1) (layer B.Cu) (net 26))
-  (segment (start 87.58 34.62) (end 86.9 35.3) (width 1) (layer B.Cu) (net 27))
-  (segment (start 90.74 34.62) (end 87.58 34.62) (width 1) (layer B.Cu) (net 27))
-  (segment (start 88.2 40.97) (end 86.93 39.7) (width 1) (layer B.Cu) (net 28))
-  (segment (start 90.74 40.97) (end 88.2 40.97) (width 1) (layer B.Cu) (net 28))
+  (segment (start 87.95 34.25) (end 86.9 35.3) (width 1) (layer B.Cu) (net 27))
+  (segment (start 90.3 34.25) (end 87.95 34.25) (width 1) (layer B.Cu) (net 27))
+  (segment (start 87.83 40.6) (end 86.93 39.7) (width 1) (layer B.Cu) (net 28))
+  (segment (start 90.3 40.6) (end 87.83 40.6) (width 1) (layer B.Cu) (net 28))
   (segment (start 81.886508 67.945) (end 83.3 67.945) (width 1) (layer B.Cu) (net 29))
   (segment (start 80.1 58.26) (end 80.1 66.158492) (width 1) (layer B.Cu) (net 29))

Commit message: PCBs updated
Parts:
- C3: footprint Capacitor_THT:C_Rect_L13.5mm_W4.0mm_P10.00mm_FKS3_FKP3_MKS4 -> Capacitor_THT:C_Disc_D4.3mm_W1.9mm_P5.00mm
- R4, R5: value 2k -> 2*k
- RV2: value 10k -> 50k
- moved C3 0.84 mm to (89.5, 48.0)
- moved RV1 0.70 mm to (89.5, 64.8)
- moved J3 0.51 mm to (89.8, 40.7)
Routing:
- net Net-(C1-Pad1): track 141.1 -> 145.2 mm
- net Net-(C3-Pad1): track 19.3 -> 18.4 mm
- net Net-(J1-Pad1): track 74.2 -> 73.5 mm
Other:
- board size 39.3 x 43.2 mm -> 38.1 x 43.2 mm
