File: schematics/visualizator_v2/visualizator_v2.kicad_pcb (KiCad board)
At the start: 2 copper layers, 95.2 x 34.3 mm, 20 parts, among them J1 5V, J2 WS2812, J3 Audio, SW1 COLOR, SW2 PATTERN, U1 ATmega328-16PU, Y1 16MHz

Commit message: PCB updated
Routing:
- net Net-(J2-Pad2): track 8.11 -> 9.32 mm
- net Net-(R3-Pad1): track 20.0 -> 19.3 mm
