File: schematics/frontpanel_v2/frontpanel.kicad_pcb (KiCad board)
At the start: 2 copper layers, 72.4 x 21.6 mm, 10 parts, among them J1 Conn_01x02_Male, J2 Conn_01x02_Male, J3 Conn_01x03_Male, J4 Conn_01x03_Male, SW1 SW_Push, SW2 SW_Push

Commit message: PCBs updated
Parts:
- removed REF** (x2): MountingHole_3.2mm_M3, MountingHole:MountingHole_3.2mm_M3
Routing:
- net Net-(J1-Pad1): track 0.28 -> 34.0 mm
- removed copper zone on B.Cu, net Net-(J1-Pad1)
Changed lines of the file:
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@@
     (thickness 1.6)
     (drawings 6)
-    (tracks 19)
+    (tracks 26)
     (zones 0)
-    (modules 10)
+    (modules 8)
     (nets 10)
   )
@@
     (last_trace_width 1)
     (trace_clearance 0.5)
-    (zone_clearance 0.6)
+    (zone_clearance 0.508)
     (zone_45_only no)
     (trace_min 0.2)
@@
     (visible_elements FFFFFF7F)
     (pcbplotparams
-      (layerselection 0x00000_fffffffe)
+      (layerselection 0x010fc_ffffffff)
       (usegerberextensions false)
       (usegerberattributes false)
       (usegerberadvancedattributes false)
       (creategerberjobfile false)
-      (excludeedgelayer false)
+      (excludeedgelayer true)
       (linewidth 0.100000)
       (plotframeref false)
@@
       (hpglpenspeed 20)
       (hpglpendiameter 15.000000)
-      (psnegative true)
+      (psnegative false)
       (psa4output false)
-      (plotreference false)
-      (plotvalue false)
+      (plotreference true)
+      (plotvalue true)
       (plotinvisibletext false)
-      (padsonsilk true)
+      (padsonsilk false)
       (subtractmaskfromsilk false)
-      (outputformat 4)
+      (outputformat 1)
       (mirror false)
-      (drillshape 2)
+      (drillshape 1)
       (scaleselection 1)
       (outputdirectory ""))
@@
     )
   )
-  (module MountingHole:MountingHole_3.2mm_M3 (layer F.Cu)
-    (at 109 119.5)
-    (descr "Mounting Hole 3.2mm, no annular, M3")
-    (tags "mounting hole 3.2mm no annular m3")
-    (attr virtual)
-    (fp_text reference REF** (at 0 -4.2) (layer F.SilkS)
-      (effects (font (size 1 1) (thickness 0.15)))
-    )
-    (fp_text value MountingHole_3.2mm_M3 (at 0 4.2) (layer F.Fab)
-      (effects (font (size 1 1) (thickness 0.15)))
-    )
-    (fp_circle (center 0 0) (end 3.45 0) (layer F.CrtYd) (width 0.05))
-    (fp_circle (center 0 0) (end 3.2 0) (layer Cmts.User) (width 0.15))
-    (fp_text user %R (at 0.3 0) (layer F.Fab)
-      (effects (font (size 1 1) (thickness 0.15)))
-    )
-    (pad 1 np_thru_hole circle (at 0 0) (size 3.2 3.2) (drill 3.2) (layers *.Cu *.Mask))
-  )
-  (module MountingHole:MountingHole_3.2mm_M3 (layer F.Cu)
-    (at 44.8 119.4)
-    (descr "Mounting Hole 3.2mm, no annular, M3")
-    (tags "mounting hole 3.2mm no annular m3")
-    (attr virtual)
-    (fp_text reference REF** (at 0 -4.2) (layer F.SilkS)
-      (effects (font (size 1 1) (thickness 0.15)))
-    )
-    (fp_text value MountingHole_3.2mm_M3 (at 0 4.2) (layer F.Fab)
-      (effects (font (size 1 1) (thickness 0.15)))
-    )
-    (fp_circle (center 0 0) (end 3.45 0) (layer F.CrtYd) (width 0.05))
-    (fp_circle (center 0 0) (end 3.2 0) (layer Cmts.User) (width 0.15))
-    (fp_text user %R (at 0.3 0) (layer F.Fab)
-      (effects (font (size 1 1) (thickness 0.15)))
-    )
-    (pad 1 np_thru_hole circle (at 0 0) (size 3.2 3.2) (drill 3.2) (layers *.Cu *.Mask))
+  (dimension 21.59 (width 0.3) (layer Dwgs.User)
+    (gr_text "21,590 mm" (at 33.46 121.285 90) (layer Dwgs.User)
+      (effects (font (size 1.5 1.5) (thickness 0.3)))
+    )
+    (feature1 (pts (xy 40.64 110.49) (xy 34.973579 110.49)))
+    (feature2 (pts (xy 40.64 132.08) (xy 34.973579 132.08)))
+    (crossbar (pts (xy 35.56 132.08) (xy 35.56 110.49)))
+    (arrow1a (pts (xy 35.56 110.49) (xy 36.146421 111.616504)))
+    (arrow1b (pts (xy 35.56 110.49) (xy 34.973579 111.616504)))
+    (arrow2a (pts (xy 35.56 132.08) (xy 36.146421 130.953496)))
+    (arrow2b (pts (xy 35.56 132.08) (xy 34.973579 130.953496)))
   )
   (dimension 72.39 (width 0.3) (layer Dwgs.User)
@@
     (arrow2b (pts (xy 40.64 137.16) (xy 41.766504 136.573579)))
   )
-  (dimension 21.59 (width 0.3) (layer Dwgs.User)
-    (gr_text "21,590 mm" (at 33.46 121.285 90) (layer Dwgs.User)
-      (effects (font (size 1.5 1.5) (thickness 0.3)))
-    )
-    (feature1 (pts (xy 40.64 110.49) (xy 34.973579 110.49)))
-    (feature2 (pts (xy 40.64 132.08) (xy 34.973579 132.08)))
-    (crossbar (pts (xy 35.56 132.08) (xy 35.56 110.49)))
-    (arrow1a (pts (xy 35.56 110.49) (xy 36.146421 111.616504)))
-    (arrow1b (pts (xy 35.56 110.49) (xy 34.973579 111.616504)))
-    (arrow2a (pts (xy 35.56 132.08) (xy 36.146421 130.953496)))
-    (arrow2b (pts (xy 35.56 132.08) (xy 34.973579 130.953496)))
-  )
   (gr_line (start 40.64 132.08) (end 40.64 110.49) (layer Edge.Cuts) (width 0.15))
   (gr_line (start 113.03 132.08) (end 40.64 132.08) (layer Edge.Cuts) (width 0.15))
   (gr_line (start 113.03 110.49) (end 113.03 132.08) (layer Edge.Cuts) (width 0.15))
   (gr_line (start 40.64 110.49) (end 113.03 110.49) (layer Edge.Cuts) (width 0.15))
-  (segment (start 81.08 113.03) (end 81.28 113.23) (width 1) (layer B.Cu) (net 1))
+  (segment (start 72.4 115.724) (end 72.4 125.7) (width 1) (layer B.Cu) (net 1))
+  (segment (start 72.4 113.2) (end 72.4 115.724) (width 1) (layer B.Cu) (net 1))
+  (segment (start 72.4 128.26) (end 71.12 129.54) (width 1) (layer B.Cu) (net 1))
+  (segment (start 72.4 125.7) (end 72.4 128.26) (width 1) (layer B.Cu) (net 1))
   (segment (start 67.39 129.46) (end 67.31 129.54) (width 1) (layer B.Cu) (net 2))
   (segment (start 67.4 129.45) (end 67.31 129.54) (width 1) (layer B.Cu) (net 2))
@@
   (segment (start 86.28 129.46) (end 86.36 129.54) (width 1) (layer B.Cu) (net 9))
   (segment (start 86.28 113.23) (end 86.28 129.46) (width 1) (layer B.Cu) (net 9))
-  (zone (net 1) (net_name "Net-(J1-Pad1)") (layer B.Cu) (hatch edge 0.508)
-    (connect_pads (clearance 0.6))
-    (min_thickness 0.254)
-    (fill yes (arc_segments 16) (thermal_gap 0.508) (thermal_bridge_width 0.508))
-    (polygon
-      (pts
-        (xy 40.775 110.5) (xy 113.1 110.5) (xy 113 132) (xy 40.7 132) (xy 40.7 110.4)
-      )
-    )
-  )
+  (segment (start 81.08 113.03) (end 81.28 113.23) (width 1) (layer B.Cu) (net 1))
+  (segment (start 81.28 113.23) (end 81.28 125.73) (width 1) (layer B.Cu) (net 1))
+  (segment (start 81.28 128.27) (end 82.55 129.54) (width 1) (layer B.Cu) (net 1))
+  (segment (start 81.28 125.73) (end 81.28 128.27) (width 1) (layer B.Cu) (net 1))
 )
